File: RFmodules/Filter/BandstopFilter7Order/BandstopFilter7Order_0402.kicad_pcb (KiCad board)
At the start: 2 copper layers, 18.5 x 7.5 mm, 16 parts, among them J1 SMA, J2 SMA

Commit message: Fix design guide issues
Other:
- net class Default: clearance 0.2 -> 0.16
- rule trace_clearance: 0.2 -> 0.16
Changed lines of the file:
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@@
     (34 B.Paste user)
     (35 F.Paste user)
-    (36 B.SilkS user hide)
+    (36 B.SilkS user)
     (37 F.SilkS user hide)
     (38 B.Mask user)
@@
   (setup
     (last_trace_width 0.25)
-    (trace_clearance 0.2)
-    (zone_clearance 0.2)
+    (trace_clearance 0.16)
+    (zone_clearance 0.1)
     (zone_45_only no)
     (trace_min 0.2)
@@
   (net 9 "Net-(C7-Pad2)")
   (net_class Default "This is the default net class."
-    (clearance 0.2)
+    (clearance 0.16)
     (trace_width 0.25)
     (via_dia 0.6)
@@
     )
   )
-  (gr_line (start 149.61108 110.40364) (end 144.89684 110.40364) (layer B.SilkS) (width 1.75))
+  (gr_line (start 150.65756 110.40364) (end 144.2212 110.40364) (layer B.SilkS) (width 1.75))
   (gr_text "Bandstop Filter 7 Order\nRevision 0.1.0 - 01/2019\ngithub.com/fgaletsee/RFLego" (at 147.3708 107.696) (layer B.SilkS)
     (effects (font (size 0.6 0.6) (thickness 0.15)) (justify mirror))
@@
   (gr_line (start 156.6418 104.14) (end 156.6418 111.6584) (layer Edge.Cuts) (width 0.1))
   (gr_line (start 138.176 104.14) (end 156.6418 104.14) (layer Edge.Cuts) (width 0.1))
+  (segment (start 140.1826 107.8992) (end 142.9766 107.8992) (width 0.61) (layer F.Cu) (net 1))
+  (segment (start 142.9766 107.8992) (end 143.9672 107.8992) (width 0.61) (layer F.Cu) (net 1))
+  (segment (start 143.9672 108.9104) (end 143.9624 108.9152) (width 0.61) (layer F.Cu) (net 1))
+  (segment (start 143.9672 107.8992) (end 143.9672 108.9104) (width 0.61) (layer F.Cu) (net 1))
   (via (at 151.892 110.8964) (size 0.6) (drill 0.3) (layers F.Cu B.Cu) (net 2))
   (via (at 148.844 110.8964) (size 0.6) (drill 0.3) (layers F.Cu B.Cu) (net 2))
   (via (at 145.923 110.8964) (size 0.6) (drill 0.3) (layers F.Cu B.Cu) (net 2))
   (via (at 143.002 110.8964) (size 0.6) (drill 0.3) (layers F.Cu B.Cu) (net 2))
-  (segment (start 140.1826 107.8992) (end 142.9766 107.8992) (width 0.61) (layer F.Cu) (net 1))
-  (segment (start 142.9766 107.8992) (end 143.9672 107.8992) (width 0.61) (layer F.Cu) (net 1))
-  (segment (start 143.9672 108.9104) (end 143.9624 108.9152) (width 0.61) (layer F.Cu) (net 1))
-  (segment (start 143.9672 107.8992) (end 143.9672 108.9104) (width 0.61) (layer F.Cu) (net 1))
   (via (at 138.938 106.5784) (size 0.6) (drill 0.3) (layers F.Cu B.Cu) (net 2))
   (via (at 139.954 106.5784) (size 0.6) (drill 0.3) (layers F.Cu B.Cu) (net 2))
@@
   (segment (start 151.8412 108.8692) (end 151.8412 109.81704) (width 0.61) (layer F.Cu) (net 9))
   (zone (net 2) (net_name GND) (layer F.Cu) (hatch edge 0.508)
-    (connect_pads yes (clearance 0.2))
+    (connect_pads yes (clearance 0.1))
     (min_thickness 0.254)
     (fill yes (arc_segments 16) (thermal_gap 0.508) (thermal_bridge_width 0.508))
@@
   )
   (zone (net 2) (net_name GND) (layer B.Cu) (hatch edge 0.508)
-    (connect_pads yes (clearance 0.2))
+    (connect_pads yes (clearance 0.1))
     (min_thickness 0.254)
     (fill yes (arc_segments 16) (thermal_gap 0.508) (thermal_bridge_width 0.508))

Commit message: Fix typos
Other:
- board text added: "Bandstop Filter 7th Order Revision 0.1.0 - 01/2019 github.com/fgaletsee/RFLego"
- board text removed: "Bandstop Filter 7 Order Revision 0.1.0 - 01/2019 github.com/fgaletsee/RFLego"
Changed lines of the file:
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@@
   (layers
     (0 F.Cu signal)
-    (31 B.Cu signal hide)
+    (31 B.Cu signal)
     (32 B.Adhes user)
     (33 F.Adhes user)
@@
     (35 F.Paste user)
     (36 B.SilkS user)
-    (37 F.SilkS user hide)
+    (37 F.SilkS user)
     (38 B.Mask user)
     (39 F.Mask user)
@@
   )
   (gr_line (start 150.65756 110.40364) (end 144.2212 110.40364) (layer B.SilkS) (width 1.75))
-  (gr_text "Bandstop Filter 7 Order\nRevision 0.1.0 - 01/2019\ngithub.com/fgaletsee/RFLego" (at 147.3708 107.696) (layer B.SilkS)
+  (gr_text "Bandstop Filter 7th Order\nRevision 0.1.0 - 01/2019\ngithub.com/fgaletsee/RFLego" (at 147.3708 107.696) (layer B.SilkS)
     (effects (font (size 0.6 0.6) (thickness 0.15)) (justify mirror))
   )

Commit message: Update board descriptions, add Bandstop elliptic filter 5th order
Other:
- board text added: "Bandstop Filter 7th Order Revision 1 - 01/2019 github.com/fgaletsee/RFLego"
- board text removed: "Bandstop Filter 7th Order Revision 0.1.0 - 01/2019 github.com/fgaletsee/RFLego"
Changed lines of the file:
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@@
   )
   (gr_line (start 150.65756 110.40364) (end 144.2212 110.40364) (layer B.SilkS) (width 1.75))
-  (gr_text "Bandstop Filter 7th Order\nRevision 0.1.0 - 01/2019\ngithub.com/fgaletsee/RFLego" (at 147.3708 107.696) (layer B.SilkS)
+  (gr_text "Bandstop Filter 7th Order\nRevision 1 - 01/2019\ngithub.com/fgaletsee/RFLego" (at 147.3708 107.696) (layer B.SilkS)
     (effects (font (size 0.6 0.6) (thickness 0.15)) (justify mirror))
   )
