File: RFmodules/Filter/Filter3Ord/Filter3Ord_1206.kicad_pcb (KiCad board)
At the start: 2 copper layers, 38.1 x 8.3 mm, 9 parts, among them J1 SMA, J2 SMA

Commit message: Update board descriptions, add Bandstop elliptic filter 5th order
Other:
- board text added: "Bandpass Filter 3th Order Revision 1 - 01/2019 github.com/fgaletsee/RFLego"
Changed lines of the file:
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@@
-(kicad_pcb (version 20171130) (host pcbnew 5.0.1)
+(kicad_pcb (version 20171130) (host pcbnew "(5.0.1-3-g963ef8bb5)")
   (general
     (thickness 1.6)
-    (drawings 6)
+    (drawings 7)
     (tracks 34)
     (zones 0)
@@
     (last_trace_width 0.2032)
     (trace_clearance 0.2032)
-    (zone_clearance 0.508)
+    (zone_clearance 0.1)
     (zone_45_only no)
     (trace_min 0.2032)
@@
       (xy -1.971615 -1.454739) (xy -1.908759 -1.469184)) (layer B.SilkS) (width 0.01))
   )
+  (gr_text "Bandpass Filter 3th Order\nRevision 1 - 01/2019\ngithub.com/fgaletsee/RFLego" (at 148.6916 104.2416) (layer B.SilkS)
+    (effects (font (size 0.75 0.75) (thickness 0.1875)) (justify left mirror))
+  )
   (gr_line (start 116.205 100.33) (end 116.205 108.585) (layer Edge.Cuts) (width 0.15))
   (gr_line (start 116.84 100.33) (end 116.205 100.33) (layer Edge.Cuts) (width 0.15))
@@
   )
   (zone (net 2) (net_name GND) (layer B.Cu) (hatch edge 0.508)
-    (connect_pads (clearance 0.508))
+    (connect_pads yes (clearance 0.1))
     (min_thickness 0.254)
     (fill yes (arc_segments 16) (thermal_gap 0.508) (thermal_bridge_width 0.508))
