File: RFmodules/Filter/Filter5OrdElliptic/Filter5OrdElLiptic.kicad_pcb (KiCad board)
At the start: 2 copper layers, 39.1 x 13.2 mm, 17 parts, among them J1 SMA, J2 SMA

Commit message: Update board descriptions, add Bandstop elliptic filter 5th order
Other:
- board text added: "Bandpass Filter Elliptic 5th Order Revision 1 - 01/2019 github.com/fgaletsee/RFLego"
- board text removed: "Bandpass Filter Elliptic 5th Order Revision 0.1.0 - 01/2019 github.com/fgaletsee/RFLego"
Changed lines of the file:
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@@
       (xy -2.549664 -1.91989) (xy -2.469928 -1.911165) (xy -2.400256 -1.919918)) (layer B.SilkS) (width 0.01))
   )
-  (gr_text "Bandpass Filter Elliptic 5th Order\nRevision 0.1.0 - 01/2019\ngithub.com/fgaletsee/RFLego" (at 134.0104 79.9338) (layer B.SilkS)
+  (gr_text "Bandpass Filter Elliptic 5th Order\nRevision 1 - 01/2019\ngithub.com/fgaletsee/RFLego" (at 134.0104 79.9338) (layer B.SilkS)
     (effects (font (size 0.75 0.75) (thickness 0.1875)) (justify left mirror))
   )
