File: RFmodules/Line/Line.kicad_pcb (KiCad board)
At the start: 2 copper layers, 48.3 x 7.6 mm, 3 parts, among them J1 SMA, J2 SMA

Commit message: Fix typos
Parts:
- moved REF** 0.23 mm to (110.1, 84.9)
Changed lines of the file:
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@@
   )
   (module Symbol:OSHW-Logo2_7.3x6mm_SilkScreen (layer B.Cu)
-    (at 110.363 84.963 180)
+    (at 110.1344 84.9376 180)
     (descr "Open Source Hardware Symbol")
     (tags "Logo Symbol OSHW")

Commit message: Update board descriptions, add Bandstop elliptic filter 5th order
Other:
- board text added: "Line Revision 1 - 01/2019 github.com/fgaletsee/RFLego"
- board text removed: "Line Revision 0.1.0 - 01/2019 github.com/fgaletsee/RFLego"
Changed lines of the file:
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@@
       (xy -2.549664 -1.91989) (xy -2.469928 -1.911165) (xy -2.400256 -1.919918)) (layer B.SilkS) (width 0.01))
   )
-  (gr_text "Line\nRevision 0.1.0 - 01/2019\ngithub.com/fgaletsee/RFLego" (at 146.05 84.836) (layer B.SilkS)
+  (gr_text "Line\nRevision 1 - 01/2019\ngithub.com/fgaletsee/RFLego" (at 146.05 84.836) (layer B.SilkS)
     (effects (font (size 0.75 0.75) (thickness 0.1875)) (justify left mirror))
   )
