File: RFmodules/Filter/Saw/433_ISM/433_ISM.kicad_pcb (KiCad board)
At the start: 2 copper layers, 14.7 x 7.9 mm, 3 parts, among them J1 SMA, J2 SMA

Commit message: Minor fixes and improvments
Routing:
- net GND: vias 4 -> 16
Other:
- board text added: "SAW Filter 3 x 3 mm Revision 1 - 01/2019 github.com/fgaletsee/RFLego"
Changed lines of the file:
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@@
-(kicad_pcb (version 20171130) (host pcbnew "(5.0.1)-4")
+(kicad_pcb (version 20171130) (host pcbnew "(5.0.1-3-g963ef8bb5)")
   (general
     (thickness 1.6)
-    (drawings 4)
-    (tracks 8)
+    (drawings 5)
+    (tracks 20)
     (zones 0)
     (modules 3)
@@
   )
   (setup
-    (last_trace_width 0.762)
+    (last_trace_width 0.2032)
     (user_trace_width 0.508)
     (user_trace_width 0.762)
     (user_trace_width 2.032)
     (trace_clearance 0.2032)
-    (zone_clearance 0.508)
+    (zone_clearance 0.1)
     (zone_45_only no)
     (trace_min 0.2032)
@@
     (pad_to_mask_clearance 0.051)
     (solder_mask_min_width 0.25)
-    (aux_axis_origin 0 0)
+    (aux_axis_origin 124.46 99.314)
+    (grid_origin 124.46 99.314)
     (visible_elements 7FFFFFFF)
     (pcbplotparams
@@
   (module RFLego_Footprint:SM3030-6 (layer F.Cu)
     (at 130.946 94.14)
-    (fp_text reference F1 (at 0.88 3.81) (layer F.SilkS)
-      (effects (font (size 1 1) (thickness 0.15)))
+    (fp_text reference F1 (at 1.134 4.412) (layer F.SilkS)
+      (effects (font (size 0.75 0.75) (thickness 0.15)))
     )
     (fp_text value SAW (at 1.27 -1.27) (layer F.Fab)
@@
     (pad 1 smd rect (at 2.032 0) (size 4.064 1.524) (layers F.Cu F.Mask)
       (net 1 "Net-(F1-Pad2)"))
+  )
+  (gr_text "SAW Filter 3 x 3 mm\nRevision 1 - 01/2019\ngithub.com/fgaletsee/RFLego" (at 131.826 95.25) (layer B.SilkS)
+    (effects (font (size 0.6 0.6) (thickness 0.15)) (justify mirror))
   )
   (gr_line (start 124.46 99.314) (end 124.46 91.44) (layer Edge.Cuts) (width 0.15))
@@
   (segment (start 137.08 95.33) (end 137.16 95.25) (width 0.762) (layer F.Cu) (net 1))
   (segment (start 133.096 95.33) (end 137.08 95.33) (width 0.762) (layer F.Cu) (net 1))
-  (via (at 130.556 98.044) (size 0.6096) (drill 0.3048) (layers F.Cu B.Cu) (net 2))
-  (via (at 132.842 98.044) (size 0.6096) (drill 0.3048) (layers F.Cu B.Cu) (net 2))
-  (via (at 130.81 92.456) (size 0.6096) (drill 0.3048) (layers F.Cu B.Cu) (net 2))
-  (via (at 132.842 92.456) (size 0.6096) (drill 0.3048) (layers F.Cu B.Cu) (net 2))
+  (via (at 134.366 94.234) (size 0.6096) (drill 0.3048) (layers F.Cu B.Cu) (net 2))
+  (via (at 134.366 96.52) (size 0.6096) (drill 0.3048) (layers F.Cu B.Cu) (net 2))
+  (via (at 134.366 93.218) (size 0.6096) (drill 0.3048) (layers F.Cu B.Cu) (net 2))
+  (via (at 134.366 97.536) (size 0.6096) (drill 0.3048) (layers F.Cu B.Cu) (net 2))
+  (via (at 133.35 93.218) (size 0.6096) (drill 0.3048) (layers F.Cu B.Cu) (net 2))
+  (via (at 132.334 93.218) (size 0.6096) (drill 0.3048) (layers F.Cu B.Cu) (net 2))
+  (via (at 131.318 93.218) (size 0.6096) (drill 0.3048) (layers F.Cu B.Cu) (net 2))
+  (via (at 130.302 93.218) (size 0.6096) (drill 0.3048) (layers F.Cu B.Cu) (net 2))
+  (via (at 133.35 97.536) (size 0.6096) (drill 0.3048) (layers F.Cu B.Cu) (net 2))
+  (via (at 132.334 97.536) (size 0.6096) (drill 0.3048) (layers F.Cu B.Cu) (net 2))
+  (via (at 131.318 97.536) (size 0.6096) (drill 0.3048) (layers F.Cu B.Cu) (net 2))
+  (via (at 130.302 97.536) (size 0.6096) (drill 0.3048) (layers F.Cu B.Cu) (net 2))
+  (via (at 129.286 93.218) (size 0.6096) (drill 0.3048) (layers F.Cu B.Cu) (net 2))
+  (via (at 129.286 94.234) (size 0.6096) (drill 0.3048) (layers F.Cu B.Cu) (net 2))
+  (via (at 129.286 96.52) (size 0.6096) (drill 0.3048) (layers F.Cu B.Cu) (net 2))
+  (via (at 129.286 97.536) (size 0.6096) (drill 0.3048) (layers F.Cu B.Cu) (net 2))
   (segment (start 126.572 95.33) (end 126.492 95.25) (width 0.762) (layer F.Cu) (net 3))
   (segment (start 130.946 95.33) (end 126.572 95.33) (width 0.762) (layer F.Cu) (net 3))
   (zone (net 2) (net_name GND) (layer F.Cu) (hatch edge 0.508)
-    (connect_pads (clearance 0.508))
+    (connect_pads yes (clearance 0.1))
     (min_thickness 0.254)
     (fill yes (arc_segments 16) (thermal_gap 0.508) (thermal_bridge_width 0.508))
@@
   )
   (zone (net 2) (net_name GND) (layer B.Cu) (hatch edge 0.508)
-    (connect_pads (clearance 0.508))
+    (connect_pads yes (clearance 0.1))
     (min_thickness 0.254)
     (fill yes (arc_segments 16) (thermal_gap 0.508) (thermal_bridge_width 0.508))
