File: RFmodules/Other/DBMixer/DBMixer.kicad_pcb (KiCad board)
At the start: 2 copper layers, 9 parts, among them J1 SMA, J2 SMA, J3 SMA, U1 T, U2 T

Commit message: Minor fixes and improvments
Parts:
- added REF**: OSHW-Logo2_7.3x6mm_SilkScreen, Symbol:OSHW-Logo2_7.3x6mm_SilkScreen, B.Cu at (129.5, 87.4)
Routing:
- net GND: vias 24 -> 50
Other:
- board outline added: 31 x 12.2 mm
- board text added: "DB Mixer"
- board text added: "DB Mixer Revision 1 - 01/2019 github.com/fgaletsee/RFLego"
