File: RFmodules/Other/DBMixer_BAT54SL/DBMixer.kicad_pcb (KiCad board)
At the start: 2 copper layers, 7 parts, among them J1 SMA, J2 SMA, J3 SMA, U1 T, U2 T

Commit message: Minor fixes and improvments
Parts:
- added REF**: OSHW-Logo2_7.3x6mm_SilkScreen, Symbol:OSHW-Logo2_7.3x6mm_SilkScreen, B.Cu at (129.5, 86.9)
Routing:
- net GND: vias 23 -> 37
Other:
- board outline added: 31 x 12.2 mm
- board text added: "DB Mixer BAT53SL"
- board text added: "DB Mixer BAT54SL Revision 1 - 01/2019 github.com/fgaletsee/RFLego"
