File: RFmodules/Other/NoiseSoruce/NoiseSoruce.kicad_pcb (KiCad board)
At the start: 2 copper layers, 47 x 7.6 mm, 20 parts, among them J1 SMA, J2 SMA, Q1 BC858

Commit message: Minor fixes and improvments
Parts:
- added REF**: OSHW-Logo2_7.3x6mm_SilkScreen, Symbol:OSHW-Logo2_7.3x6mm_SilkScreen, B.Cu at (155.2, 107.7)
- moved D2 0.18 mm to (152.0, 109.7)
- renumbered J1 to OUT
Routing:
- net Net-(C6-Pad1): track 20.0 -> 20.8 mm
- net GND: vias 20 -> 43
Other:
- board text added: "Noise Source 100 MHz - 2.5 GHz Revision 1 - 01/2019 github.com/fgaletsee/RFLego"
- board text removed: "out"
