File: KicadTemplate/RFLegoTemplate/RFLegoTemplate.kicad_pcb (KiCad board)
At the start: 2 copper layers, 0 parts

Commit message: Add thin 50 Ohm track
Other:
- net class 50 Ohm thin added: clearance 0.1524, trace_width 1.0922, via_dia 0.6096, via_drill 0.3048
- rule trace_min: 0.2032 -> 0.1524
Changed lines of the file:
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@@
-(kicad_pcb (version 20171130) (host pcbnew 5.0.1)
+(kicad_pcb (version 20171130) (host pcbnew "(5.0.1-3-g963ef8bb5)")
   (general
     (thickness 1.6)
@@
     (zone_clearance 0.508)
     (zone_45_only no)
-    (trace_min 0.2032)
+    (trace_min 0.1524)
     (segment_width 0.2)
     (edge_width 0.15)
@@
     (via_dia 0.6096)
     (via_drill 0.3048)
+    (uvia_dia 0.3)
+    (uvia_drill 0.1)
+    (diff_pair_gap 0.2032)
+    (diff_pair_width 0.2032)
+  )
+  (net_class "50 Ohm thin" ""
+    (clearance 0.1524)
+    (trace_width 1.0922)
+    (via_dia 0.6096)
+    (via_drill 0.3048)

Commit message: Update PCB design rules based on https://chemandy.com/calculators/coplanar-waveguide-with-ground-calculator.htm
Other:
- net class 50 Ohm thin: clearance 0.1524 -> 0.1778; trace_width 1.0922 -> 1.2192; via_dia 0.6096 -> 0.7; via_drill 0.3048 -> 0.35
- net class 50Ohm: clearance 0.37 -> 0.32004; trace_width 1.8 -> 1.778; via_dia 0.6096 -> 0.7; via_drill 0.3048 -> 0.35
- net class Default: clearance 0.2032 -> 0.2286; trace_width 0.2032 -> 0.2286; via_dia 0.6096 -> 0.7; via_drill 0.3048 -> 0.35
- rule trace_clearance: 0.2032 -> 0.2286
- rule trace_min: 0.1524 -> 0.2032
Changed lines of the file:
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@@
   )
   (setup
-    (last_trace_width 0.2032)
-    (trace_clearance 0.2032)
+    (last_trace_width 0.2286)
+    (trace_clearance 0.2286)
     (zone_clearance 0.508)
     (zone_45_only no)
-    (trace_min 0.1524)
+    (trace_min 0.2032)
     (segment_width 0.2)
     (edge_width 0.15)
-    (via_size 0.6096)
-    (via_drill 0.3048)
+    (via_size 0.7)
+    (via_drill 0.35)
     (via_min_size 0.6096)
     (via_min_drill 0.3048)
@@
   (net 0 "")
   (net_class Default "This is the default net class."
-    (clearance 0.2032)
-    (trace_width 0.2032)
-    (via_dia 0.6096)
-    (via_drill 0.3048)
+    (clearance 0.2286)
+    (trace_width 0.2286)
+    (via_dia 0.7)
+    (via_drill 0.35)
     (uvia_dia 0.3)
     (uvia_drill 0.1)
@@
   )
   (net_class "50 Ohm thin" ""
-    (clearance 0.1524)
-    (trace_width 1.0922)
-    (via_dia 0.6096)
-    (via_drill 0.3048)
+    (clearance 0.1778)
+    (trace_width 1.2192)
+    (via_dia 0.7)
+    (via_drill 0.35)
     (uvia_dia 0.3)
     (uvia_drill 0.1)
@@
   )
   (net_class 50Ohm ""
-    (clearance 0.37)
-    (trace_width 1.8)
-    (via_dia 0.6096)
-    (via_drill 0.3048)
+    (clearance 0.32004)
+    (trace_width 1.778)
+    (via_dia 0.7)
+    (via_drill 0.35)
     (uvia_dia 0.3)
     (uvia_drill 0.1)

Commit message: Update KiCAD template based on new PCB base layout
Parts:
- added H1: MountingHole_Pad, MountingHole:MountingHole_2.2mm_M2_Pad_Via, F.Cu at (102.2, 102.2)
- added H2: MountingHole_Pad, MountingHole:MountingHole_2.2mm_M2_Pad_Via, F.Cu at (102.2, 115.8)
- added H3: MountingHole_Pad, MountingHole:MountingHole_2.2mm_M2_Pad_Via, F.Cu at (129.8, 102.2)
- added H4: MountingHole_Pad, MountingHole:MountingHole_2.2mm_M2_Pad_Via, F.Cu at (129.8, 115.8)
- added J1: SMA, RFLego_Footprint:SMA_Edge, F.Cu at (100.0, 109.0)
- added J2: SMA, RFLego_Footprint:SMA_Edge, F.Cu at (128.0, 109.0)
- added REF**: OSHW-Logo2_9.8x8mm_SilkScreen, Symbol:OSHW-Logo2_9.8x8mm_SilkScreen, B.Cu at (109.5, 113.2)
Routing:
- net GND: vias 0 -> 66
- added copper zone on B.Cu, net GND
- added copper zone on F.Cu, net GND
Other:
- board outline added: 32 x 18 mm
- net class 50 Ohm thin: clearance 0.1778 -> 0.19; trace_width 1.2192 -> 1; via_drill 0.35 -> 0.4
- net class 50Ohm: clearance 0.32004 -> 0.32; trace_width 1.778 -> 1.5; via_drill 0.35 -> 0.4
- net class Default: clearance 0.2286 -> 0.2; trace_width 0.2286 -> 0.22; via_drill 0.35 -> 0.4
- rule trace_clearance: 0.2286 -> 0.2
- rule trace_min: 0.2032 -> 0.2
- rule via_min_drill: 0.3048 -> 0.3
- rule via_min_size: 0.6096 -> 0.6
- board text added: "Line Revision 1 - 02/2019 github.com/fgaletsee/RFLego"
