File: RFmodules/Filter/Saw/433_SAW/433_SAW.kicad_pcb (KiCad board)
At the start: 2 copper layers, 32 x 18 mm, 10 parts, among them J1 SMA, J2 SMA

Commit message: SAW and PI Module updated!
Parts:
- removed R1, R2, R3: R, Resistor_SMD:R_0805_2012Metric
- added F1: SF2136E, RFLego_Footprint:SM3030-6, F.Cu at (115.2, 107.8)
Other:
- board text added: "SAW Revision 1 - 02/2019 github.com/fgaletsee/RFLego"
- board text removed: "PI Revision 1 - 02/2019 github.com/fgaletsee/RFLego"
