File: RFmodules/Other/Balun/Balun.kicad_pcb (KiCad board)
At the start: 2 copper layers, 32 x 18 mm, 7 parts, among them J1 SMA, J2 SMA

Commit message: Update Balun to use new module template
Parts:
- removed the REF** at (109.5, 113.2)
- added J4: SMA, RFLego_Footprint:SMA_Edge, F.Cu at (120.0, 118.0)
- added REF**: OSHW-Logo2_9.8x8mm_SilkScreen, Symbol:OSHW-Logo2_9.8x8mm_SilkScreen, B.Cu at (0.00, 96.5)
- added REF**: OSHW-Logo2_9.8x8mm_SilkScreen, Symbol:OSHW-Logo2_9.8x8mm_SilkScreen, B.Cu at (110.5, 113.0)
- added U1: T, RFLego_Footprint:Coilcraft_WBC_HandSolder, F.Cu at (119.9, 109.0)
- moved J2 9.39 mm to (120.0, 104.0), turned to 90 degrees
Connections:
- J1 pad 1: (no net) -> Net-(J1-Pad1)
- J2 pad 1: (no net) -> Net-(J2-Pad1)
Routing:
- net Net-(J1-Pad1): track 0.00 -> 14.7 mm
- net Net-(J2-Pad1): track 0.00 -> 7.00 mm
- net Net-(J4-Pad1): track 0.00 -> 3.95 mm
- net GND: vias 66 -> 59
Other:
- board text added: "Balun Revision 1 - 02/2019 github.com/fgaletsee/RFLego"
- board text removed: "Line Revision 1 - 02/2019 github.com/fgaletsee/RFLego"
