File: RFmodules/Other/Balun/Balun.sch (KiCad schematic (older format))
At the start: 4 parts, among them J1 SMA, J2 SMA, J3 SMA, U1 T

Commit message: Update Balun to use new module template
Parts:
- removed J3: SMA, RFLego_Footprint:SMA_Edge, symbol RFLego_Schematic:SMA
- added H1, H2, H3, H4: MountingHole_Pad, MountingHole:MountingHole_2.2mm_M2_Pad_Via, symbol Mechanical:MountingHole_Pad
- added J3: RF_Shield_One_Piece, symbol Device:RF_Shield_One_Piece
- added J4: SMA, RFLego_Footprint:SMA_Edge, symbol RFLego_Schematic:SMA
Connections:
- net labels removed: out_N, out_Px
Other:
- note added: "Do not edit"
- note added: "If possible, use these two connecters\nfor a compatible netlist used in our\nPCB template."
