File: RFmodules/Aktive/EigenePA/EigenePA.kicad_pcb (KiCad board)
At the start: 2 copper layers, 32 x 18 mm, 22 parts, among them J1 SMA, J2 SMA, Q1 BC817

Commit message: Edit B Silk Label
Other:
- board text added: "BC817 RF-PA Revision 1 - 02/2019 github.com/fgaletsee/RFLego"
- board text removed: "Line Revision 1 - 02/2019 github.com/fgaletsee/RFLego"
Changed lines of the file:
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@@
     (34 B.Paste user)
     (35 F.Paste user)
-    (36 B.SilkS user hide)
+    (36 B.SilkS user)
     (37 F.SilkS user)
     (38 B.Mask user hide)
@@
   )
   (setup
-    (last_trace_width 0.508)
+    (last_trace_width 0.22)
     (user_trace_width 0.254)
     (user_trace_width 0.381)
@@
   (gr_line (start 132 111.73) (end 132 115.75) (layer F.Mask) (width 2))
   (gr_line (start 100 111.73) (end 100 115.75) (layer F.Mask) (width 2))
-  (gr_text "Line\nRevision 1 - 02/2019\ngithub.com/fgaletsee/RFLego" (at 127.75 106.25) (layer B.SilkS)
+  (gr_text "BC817 RF-PA \nRevision 1 - 02/2019\ngithub.com/fgaletsee/RFLego" (at 127.75 106.25) (layer B.SilkS)
     (effects (font (size 1 1) (thickness 0.25)) (justify left mirror))
   )

Commit message: Layout angepasst
Parts:
- moved R2 4.50 mm to (111.4, 110.6)
- moved R4 1.32 mm to (113.9, 113.7)
- moved R5 1.32 mm to (120.7, 112.7)
- moved C3 1.32 mm to (116.8, 112.7)
Routing:
- net Net-(C1-Pad1): track 15.5 -> 10.5 mm
- net Net-(C3-Pad2): track 4.69 -> 3.43 mm
Changed lines of the file:
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@@
-(kicad_pcb (version 20171130) (host pcbnew "(5.0.1)-4")
+(kicad_pcb (version 20171130) (host pcbnew "(5.1.4)-1")
   (general
     (thickness 1.6)
@@
   )
   (setup
-    (last_trace_width 0.22)
+    (last_trace_width 0.508)
     (user_trace_width 0.254)
     (user_trace_width 0.381)
@@
     (zone_45_only no)
     (trace_min 0.2)
-    (segment_width 0.15)
-    (edge_width 0.15)
     (via_size 0.7)
     (via_drill 0.4)
@@
     (uvia_min_size 0.2)
     (uvia_min_drill 0.1)
+    (edge_width 0.15)
+    (segment_width 0.15)
     (pcb_text_width 0.3)
     (pcb_text_size 1.5 1.5)
@@
     (uvia_dia 0.3)
     (uvia_drill 0.1)
+    (diff_pair_width 0.2)
     (diff_pair_gap 0.2)
-    (diff_pair_width 0.2)
     (add_net GND)
     (add_net "Net-(C1-Pad1)")
@@
     (uvia_dia 0.3)
     (uvia_drill 0.1)
+    (diff_pair_width 0.2)
     (diff_pair_gap 0.2)
-    (diff_pair_width 0.2)
   )
   (net_class 50Ohm ""
@@
     (uvia_dia 0.3)
     (uvia_drill 0.1)
+    (diff_pair_width 0.2)
     (diff_pair_gap 0.2)
-    (diff_pair_width 0.2)
   )
   (module MountingHole:MountingHole_2.2mm_M2_Pad_Via (layer F.Cu)
@@
   )
   (module Capacitor_SMD:C_0603_1608Metric_Pad1.05x0.95mm_HandSolder (layer F.Cu)
-    (at 116.623 113.97 180)
+    (at 116.823 112.67 180)
     (descr "Capacitor SMD 0603 (1608 Metric), square (rectangular) end terminal, IPC_7351 nominal with elongated pad for handsoldering. (Body size source: http://www.tortai-tech.com/upload/download/2011102023233369053.pdf), generated with kicad-footprint-generator")
     (tags "capacitor handsolder")
@@
   )
   (module Resistor_SMD:R_0603_1608Metric_Pad1.05x0.95mm_HandSolder (layer F.Cu)
-    (at 109.906 114.873 270)
+    (at 111.4 110.625 270)
     (descr "Resistor SMD 0603 (1608 Metric), square (rectangular) end terminal, IPC_7351 nominal with elongated pad for handsoldering. (Body size source: http://www.tortai-tech.com/upload/download/2011102023233369053.pdf), generated with kicad-footprint-generator")
     (tags "resistor handsolder")
@@
   )
   (module Resistor_SMD:R_0603_1608Metric_Pad1.05x0.95mm_HandSolder (layer F.Cu)
-    (at 113.716 114.986 270)
+    (at 113.916 113.686 270)
     (descr "Resistor SMD 0603 (1608 Metric), square (rectangular) end terminal, IPC_7351 nominal with elongated pad for handsoldering. (Body size source: http://www.tortai-tech.com/upload/download/2011102023233369053.pdf), generated with kicad-footprint-generator")
     (tags "resistor handsolder")
@@
   )
   (module Resistor_SMD:R_0603_1608Metric_Pad1.05x0.95mm_HandSolder (layer F.Cu)
-    (at 120.461 113.97)
+    (at 120.661 112.67)
     (descr "Resistor SMD 0603 (1608 Metric), square (rectangular) end terminal, IPC_7351 nominal with elongated pad for handsoldering. (Body size source: http://www.tortai-tech.com/upload/download/2011102023233369053.pdf), generated with kicad-footprint-generator")
     (tags "resistor handsolder")
@@
   (via (at 131.5 113) (size 0.7) (drill 0.4) (layers F.Cu B.Cu) (net 1))
   (via (at 131.5 105) (size 0.7) (drill 0.4) (layers F.Cu B.Cu) (net 1))
-  (segment (start 109.906 112.446) (end 109.906 113.998) (width 0.508) (layer F.Cu) (net 2))
   (segment (start 111.43 107.366) (end 110.16 108.636) (width 0.508) (layer F.Cu) (net 2))
   (segment (start 112.079 107.366) (end 111.43 107.366) (width 0.508) (layer F.Cu) (net 2))
   (segment (start 107.62 108.636) (end 107.366 108.89) (width 0.508) (layer F.Cu) (net 2))
   (segment (start 110.16 108.636) (end 107.62 108.636) (width 0.508) (layer F.Cu) (net 2))
-  (segment (start 110.16 112.192) (end 109.906 112.446) (width 0.508) (layer F.Cu) (net 2))
-  (segment (start 110.348 109.464) (end 110.16 109.652) (width 0.508) (layer F.Cu) (net 2))
-  (segment (start 114.764 109.464) (end 110.348 109.464) (width 0.508) (layer F.Cu) (net 2))
-  (segment (start 110.16 108.636) (end 110.16 109.652) (width 0.508) (layer F.Cu) (net 2))
-  (segment (start 110.16 109.652) (end 110.16 112.192) (width 0.508) (layer F.Cu) (net 2))
+  (segment (start 111.686 109.464) (end 111.4 109.75) (width 0.508) (layer F.Cu) (net 2))
+  (segment (start 114.764 109.464) (end 111.686 109.464) (width 0.508) (layer F.Cu) (net 2))
+  (segment (start 110.286 108.636) (end 111.4 109.75) (width 0.508) (layer F.Cu) (net 2))
+  (segment (start 110.16 108.636) (end 110.286 108.636) (width 0.508) (layer F.Cu) (net 2))
   (segment (start 102.142 108.89) (end 102.032 109) (width 0.508) (layer F.Cu) (net 3))
   (segment (start 105.616 108.89) (end 102.142 108.89) (width 0.508) (layer F.Cu) (net 3))
   (segment (start 111.458 105.588) (end 110.16 106.886) (width 0.508) (layer F.Cu) (net 4))
   (segment (start 111.966 105.588) (end 111.458 105.588) (width 0.508) (layer F.Cu) (net 4))
-  (segment (start 117.498 113.97) (end 119.586 113.97) (width 0.508) (layer F.Cu) (net 5))
-  (segment (start 114.764 111.364) (end 114.764 113.938) (width 0.508) (layer F.Cu) (net 6))
-  (segment (start 114.591 114.111) (end 113.716 114.111) (width 0.508) (layer F.Cu) (net 6))
-  (segment (start 114.764 113.938) (end 114.591 114.111) (width 0.508) (layer F.Cu) (net 6))
-  (segment (start 114.796 113.97) (end 115.748 113.97) (width 0.508) (layer F.Cu) (net 6))
-  (segment (start 114.764 113.938) (end 114.796 113.97) (width 0.508) (layer F.Cu) (net 6))
+  (segment (start 117.698 112.67) (end 119.786 112.67) (width 0.508) (layer F.Cu) (net 5))
+  (segment (start 114.764 112.272) (end 114.75 112.286) (width 0.508) (layer F.Cu) (net 6))
+  (segment (start 114.764 111.364) (end 114.764 112.272) (width 0.508) (layer F.Cu) (net 6))
+  (segment (start 114.75 112.286) (end 114.75 112.7) (width 0.508) (layer F.Cu) (net 6))
+  (segment (start 114.639 112.811) (end 113.916 112.811) (width 0.508) (layer F.Cu) (net 6))
+  (segment (start 114.75 112.7) (end 114.639 112.811) (width 0.508) (layer F.Cu) (net 6))
+  (segment (start 114.78 112.67) (end 115.948 112.67) (width 0.508) (layer F.Cu) (net 6))
+  (segment (start 114.75 112.7) (end 114.78 112.67) (width 0.508) (layer F.Cu) (net 6))
   (segment (start 116.51 110.16) (end 116.764 110.414) (width 0.508) (layer F.Cu) (net 7))
   (segment (start 116.51 107.039) (end 116.51 110.16) (width 0.508) (layer F.Cu) (net 7))
